Commit message: feat: added initial support for gazebo

File: rbt08pkg/urdf/rbt10.urdf (robot description, URDF)
Before this commit: robot rbt10, 10 links, 9 joints
Links:
- link table_camera_link: geometry collision box size=.05 .05 .05; visual box size=.05 .05 .05

Commit message: Add RGB-D camera pipeline and YOLO environment

File: rbt08pkg/urdf/rbt10.urdf (robot description, URDF)
Before this commit: robot rbt10, 10 links, 9 joints
Joints:
- joint table_camera_joint: origin xyz=1.0 0.4 0.2 rpy=0 0 3.6652 -> xyz=0.55 1.35 1.55 rpy=0 0.2846566951 -1.2120256565
- joint table_camera_optical_joint: origin xyz=0 0 0 rpy=-1.5707 0 -1.5707 -> xyz=0 0 0 rpy=-1.5707963267948966 0 -1.5707963267948966

Commit message: feat: added HSV pear segmentation

File: rbt08pkg/urdf/rbt10.urdf (robot description, URDF)
Before this commit: robot rbt10, 10 links, 9 joints
Joints:
- joint table_camera_joint: origin xyz=0.55 1.35 1.55 rpy=0 0.2846566951 -1.2120256565 -> xyz=0.15 -0.55 1.75 rpy=0 0.3323335118 1.0040671093
